File: hardware/comms_module/Communications Board.sch (EAGLE design)
At the start: 68 parts, among them U1 Value, U2 STC3115, X2 USB-MICROB, Y1 32.768kHz, Y2 24MHz

Commit message: Nearly complete routing. Add programming interface.
Parts:
- added D1: Green, SparkFun-LED:LED1206
- added D2: Red, SparkFun-LED:LED1206
- added JP1: AVR-JTAG-10, avr-7:AVR-JTAG-10
- added R10, R20: 500, SparkFun-Passives:RESISTOR0603-RES
- added S1: (no value), Capstone Library:SWITCH-SPDT
- C8: value (none) -> 1uF
Connections:
- removed net AGND: JP8.5
- removed net BATT_ALARM: U2.ALM
- removed net JTAG_TDI: U1.DIO_6
- removed net JTAG_TDO: U1.DIO_5
- removed net N$25: JP8.9
- removed net N$26: JP8.8
- removed net N$27: JP8.6
- removed net N$28: JP8.3
- removed net N$29: JP8.1
- removed net TMR: U$2.TMR
- new net /SYSDISBL_PF: R14.1, R15.2, U$6G$2.G
- new net N$14: D1.C, R10.1
- new net N$16: D2.C, R20.1
- new net N$6: D2.A, S1.S
- new net PROG_VCC: D1.A, JP1.7, S1.P
- net +1V3: now also U1.DIO_13; no longer U1.DIO_9
- net /SYSDISBL: no longer R14.1, R15.2, U$6G$2.G
- net BANDAGE_A_0: now also JP8.6, U1.DIO_9; no longer U1.DIO_10
- net BANDAGE_A_1: now also JP8.3
- net BANDAGE_A_2: now also JP8.8
- net BANDAGE_A_3: now also JP8.1
- net BANDAGE_A_4: now also JP8.9
- net CONN_STATE_RD: now also U1.DIO_10; no longer U1.DIO_12
- net GND: now also JP1.10, JP1.2, JP8.5, R10.2, R20.2
- net JTAG_TCKC: now also JP1.1
- net JTAG_TSMC: now also JP1.5
- net MCU_RST: now also JP1.6; no longer U2.RSTIO
- net SCL: now also U1.DIO_7; no longer U1.DIO_14
- net SDA: now also U1.DIO_8; no longer U1.DIO_13
- net VCC: now also JP1.4
- net VSENSE_0: now also U1.DIO_14; no longer U1.DIO_7
- net VSENSE_1: now also U1.DIO_12; no longer U1.DIO_8
- net V_PREBUCK: now also S1.O
Other:
- note added: "JTAG Programmer Interface"
