File: hardware/bandage_module/Bandage FPC.sch (EAGLE design)
At the start: 14 parts

Commit message: Add remaining components and start board layout.
Changed lines of the file:
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@@
 <instance part="H1" gate="G$1" x="101.6" y="55.88" rot="R90"/>
 <instance part="H2" gate="G$1" x="96.52" y="53.34" rot="R90"/>
-<instance part="H3" gate="G$1" x="160.02" y="48.26" rot="R90"/>
-<instance part="H4" gate="G$1" x="147.32" y="40.64" rot="R270"/>
+<instance part="H3" gate="G$1" x="147.32" y="50.8" rot="R90"/>
+<instance part="H4" gate="G$1" x="154.94" y="48.26" rot="R90"/>
 <instance part="H5" gate="G$1" x="106.68" y="40.64" rot="R270"/>
 <instance part="H6" gate="G$1" x="91.44" y="50.8" rot="R90"/>
@@
 <pinref part="JP1" gate="G$1" pin="8"/>
 <pinref part="H4" gate="G$1" pin="P$1"/>
-<wire x1="124.46" y1="45.72" x2="147.32" y2="45.72" width="0.1524" layer="91"/>
-<wire x1="147.32" y1="45.72" x2="147.32" y2="43.18" width="0.1524" layer="91"/>
+<wire x1="124.46" y1="45.72" x2="154.94" y2="45.72" width="0.1524" layer="91"/>
 </segment>
 </net>
@@
 <segment>
 <pinref part="JP1" gate="G$1" pin="6"/>
-<wire x1="124.46" y1="48.26" x2="157.48" y2="48.26" width="0.1524" layer="91"/>
-<wire x1="157.48" y1="48.26" x2="157.48" y2="45.72" width="0.1524" layer="91"/>
+<wire x1="124.46" y1="48.26" x2="147.32" y2="48.26" width="0.1524" layer="91"/>
 <pinref part="H3" gate="G$1" pin="P$1"/>
-<wire x1="157.48" y1="45.72" x2="160.02" y2="45.72" width="0.1524" layer="91"/>
-</segment>
-</net>
+</segment>
+</net>

Commit message: Adding final draft of FPC
Parts:
- added JP2: (no value), SparkFun-Connectors:M06LOCK
- JP1: device SparkFun-Connectors:M05X2NO_SILK -> SparkFun-Connectors:M06LOCK
Connections:
- net +3V3: now also JP1.1, JP1.2, JP2.6, U$1.A0, U$1.A1, U$1.A2; no longer JP1.10
- net AGND: now also JP2.3; no longer JP1.5
- net GND: now also JP2.4; no longer JP1.7, U$1.A0, U$1.A1, U$1.A2
- net N$2: now also JP2.5; no longer JP1.1
- net N$3: now also JP2.2; no longer JP1.8
- net N$4: now also JP1.4; no longer JP1.6
- net N$5: now also JP2.1; no longer JP1.9
- net SCL: now also JP1.6; no longer JP1.2
- net SDA: now also JP1.5; no longer JP1.4
